File: DBUS.kicad_sch (KiCad schematic)
At the start: 5 parts, among them Q1 S8050, U8 CH340E

Commit message: New PCB design and single panel to SMT
Parts:
- removed Q1: S8050, Package_TO_SOT_SMD:SOT-23, symbol Transistor_BJT:S8050
- added Q1: S8050, Package_TO_SOT_SMD:SOT-23, symbol Device:Q_NPN_BEC
Connections:
- net DBus: now also Q1.1 (B)
- net GND: now also Q1.2 (E)
- net at R11.2, U8.9 (RXD): now also Q1.3 (C)
Changed lines of the file:
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@@
     (effects (font (size 1.27 1.27)) (justify left))
-  )
-  (symbol (lib_id "Transistor_BJT:S8050") (at 154.94 93.218 0) (mirror y) (unit 1)
-    (in_bom yes) (on_board yes)
-    (property "Reference" "Q1" (id 0) (at 150.876 89.916 0)
-      (effects (font (size 1.27 1.27)) (justify left))
-    )
-    (property "Value" "S8050" (id 1) (at 150.876 97.536 0)
-      (effects (font (size 1.27 1.27)) (justify left))
-    )
-    (property "Footprint" "Package_TO_SOT_SMD:SOT-23" (id 2) (at 149.86 95.123 0)
-      (effects (font (size 1.27 1.27) italic) (justify left) hide)
-    )
-    (property "Datasheet" "http://www.unisonic.com.tw/datasheet/S8050.pdf" (id 3) (at 154.94 93.218 0)
-      (effects (font (size 1.27 1.27)) (justify left) hide)
-    )
-    (pin "1")
-    (pin "2")
-    (pin "3")
   )
   (symbol (lib_id "Device:C_Small") (at 107.696 87.376 0) (mirror y) (unit 1)
@@
     (pin "1")
   )
+  (symbol (lib_id "Device:Q_NPN_BEC") (at 154.94 93.218 0) (mirror y) (unit 1)
+    (in_bom yes) (on_board yes) (fields_autoplaced)
+    (property "Reference" "Q1" (id 0) (at 150.0886 92.3095 0)
+      (effects (font (size 1.27 1.27)) (justify left))
+    )
+    (property "Value" "S8050" (id 1) (at 150.0886 95.0846 0)
+      (effects (font (size 1.27 1.27)) (justify left))
+    )
+    (property "Footprint" "Package_TO_SOT_SMD:SOT-23" (id 2) (at 149.86 90.678 0)
+      (effects (font (size 1.27 1.27)) hide)
+    )
+    (property "Datasheet" "~" (id 3) (at 154.94 93.218 0)
+      (effects (font (size 1.27 1.27)) hide)
+    )
+    (pin "1")
+    (pin "2")
+    (pin "3")
+  )
   (symbol (lib_id "power:GND") (at 152.4 106.172 0) (unit 1)
