File: STM2_CAN.kicad_sch (KiCad schematic)
At the start: 18 parts, among them J7 Conn_01x04, U4 STM32F072C8Tx, U5 TJA1051T-3

Commit message: New PCB design and single panel to SMT
Parts:
- removed J7: Conn_01x04, Connector_JST:JST_GH_BM04B-GHS-TBT_1x04-1MP_P1.25mm_Vertical, symbol Connector_Generic:Conn_01x04
Connections:
- net SWCLK: no longer names the net of U4.37 (PA14)
- net SWDIO: no longer names the net of U4.34 (PA13)
- net USB_DM renamed USB_D-
- net USB_DP renamed USB_D+
- no-connect marks 29 -> 31
Changed lines of the file:
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@@
   (no_connect (at 60.96 105.664))
   (no_connect (at 60.96 92.964))
+  (no_connect (at 93.98 110.744))
+  (no_connect (at 93.98 113.284))
   (no_connect (at 60.96 110.744))
   (no_connect (at 60.96 70.104))
@@
     (stroke (width 0) (type default) (color 0 0 0 0))
   )
-  (wire (pts (xy 120.142 102.362) (xy 120.142 101.6))
-    (stroke (width 0) (type default) (color 0 0 0 0))
-  )
   (wire (pts (xy 118.364 67.31) (xy 118.364 69.596))
     (stroke (width 0) (type default) (color 0 0 0 0))
@@
     (stroke (width 0) (type default) (color 0 0 0 0))
   )
-  (wire (pts (xy 120.142 93.98) (xy 121.666 93.98))
-    (stroke (width 0) (type default) (color 0 0 0 0))
-  )
   (wire (pts (xy 79.502 172.974) (xy 79.502 175.26))
     (stroke (width 0) (type default) (color 0 0 0 0))
@@
     (stroke (width 0) (type default) (color 0 0 0 0))
   )
-  (wire (pts (xy 120.142 101.6) (xy 121.666 101.6))
-    (stroke (width 0) (type default) (color 0 0 0 0))
-  )
   (wire (pts (xy 73.66 120.904) (xy 73.66 123.698))
-    (stroke (width 0) (type default) (color 0 0 0 0))
-  )
-  (wire (pts (xy 120.142 92.202) (xy 120.142 93.98))
     (stroke (width 0) (type default) (color 0 0 0 0))
   )
@@
     (effects (font (size 1.27 1.27)) (justify right bottom))
   )
-  (label "SWCLK" (at 121.666 99.06 180)
-    (effects (font (size 1.27 1.27)) (justify right bottom))
-  )
-  (label "SWDIO" (at 93.98 110.744 0)
-    (effects (font (size 1.27 1.27)) (justify left bottom))
-  )
   (label "CAN_TX" (at 106.68 158.242 180)
     (effects (font (size 1.27 1.27)) (justify right bottom))
@@
     (effects (font (size 1.27 1.27)) (justify left bottom))
   )
-  (label "SWDIO" (at 121.666 96.52 180)
-    (effects (font (size 1.27 1.27)) (justify right bottom))
-  )
-  (label "SWCLK" (at 93.98 113.284 0)
-    (effects (font (size 1.27 1.27)) (justify left bottom))
-  )
   (label "LED2" (at 93.98 80.264 0)
     (effects (font (size 1.27 1.27)) (justify left bottom))
@@
     (effects (font (size 1.27 1.27)) (justify left))
   )
-  (hierarchical_label "USB_DP" (shape bidirectional) (at 93.98 108.204 0)
+  (hierarchical_label "USB_D+" (shape bidirectional) (at 93.98 108.204 0)
     (effects (font (size 1.27 1.27)) (justify left))
   )
@@
     (effects (font (size 1.27 1.27)) (justify left))
   )
-  (hierarchical_label "USB_DM" (shape bidirectional) (at 93.98 105.664 0)
+  (hierarchical_label "USB_D-" (shape bidirectional) (at 93.98 105.664 0)
     (effects (font (size 1.27 1.27)) (justify left))
   )
@@
     )
     (property "Datasheet" "" (id 3) (at 60.452 40.894 0)
-      (effects (font (size 1.27 1.27)) hide)
-    )
-    (pin "1")
-  )
-  (symbol (lib_id "power:GND") (at 120.142 102.362 0) (unit 1)
-    (in_bom yes) (on_board yes) (fields_autoplaced)
-    (property "Reference" "#PWR038" (id 0) (at 120.142 108.712 0)
-      (effects (font (size 1.27 1.27)) hide)
-    )
-    (property "Value" "GND" (id 1) (at 122.047 104.111 0)
-      (effects (font (size 1.27 1.27)) (justify left))
-    )
-    (property "Footprint" "" (id 2) (at 120.142 102.362 0)
-      (effects (font (size 1.27 1.27)) hide)
-    )
-    (property "Datasheet" "" (id 3) (at 120.142 102.362 0)
       (effects (font (size 1.27 1.27)) hide)
     )
@@
     (pin "2")
   )
-  (symbol (lib_id "power:VCC") (at 120.142 92.202 0) (unit 1)
-    (in_bom yes) (on_board yes) (fields_autoplaced)
-    (property "Reference" "#PWR037" (id 0) (at 120.142 96.012 0)
-      (effects (font (size 1.27 1.27)) hide)
-    )
-    (property "Value" "VCC" (id 1) (at 120.142 88.5975 0))
-    (property "Footprint" "" (id 2) (at 120.142 92.202 0)
-      (effects (font (size 1.27 1.27)) hide)
-    )
-    (property "Datasheet" "" (id 3) (at 120.142 92.202 0)
-      (effects (font (size 1.27 1.27)) hide)
-    )
-    (pin "1")
-  )
   (symbol (lib_id "Device:R_Small") (at 134.366 163.322 0) (unit 1)
     (in_bom yes) (on_board yes)
@@
     (pin "1")
   )
-  (symbol (lib_id "Connector_Generic:Conn_01x04") (at 126.746 96.52 0) (unit 1)
-    (in_bom yes) (on_board yes) (fields_autoplaced)
-    (property "Reference" "J7" (id 0) (at 128.778 98.269 0)
-      (effects (font (size 1.27 1.27)) (justify left))
-    )
-    (property "Value" "Conn_01x04" (id 1) (at 126.746 91.5186 0)
-      (effects (font (size 1.27 1.27)) hide)
-    )
-    (property "Footprint" "Connector_JST:JST_GH_BM04B-GHS-TBT_1x04-1MP_P1.25mm_Vertical" (id 2) (at 126.746 96.52 0)
-      (effects (font (size 1.27 1.27)) hide)
-    )
-    (property "Datasheet" "~" (id 3) (at 126.746 96.52 0)
-      (effects (font (size 1.27 1.27)) hide)
-    )
-    (pin "1")
-    (pin "2")
-    (pin "3")
-    (pin "4")
-  )
   (symbol (lib_id "Device:LED") (at 53.848 170.18 90) (unit 1)
