File: USB2XXX.kicad_sch (KiCad schematic)
At the start: 12 parts, among them J1 Conn_01x04, J2 Conn_01x03, J3 Conn_01x03, J4 Conn_01x02, J5 Conn_01x02

Commit message: New PCB design and single panel to SMT
Parts:
- J1: footprint Connector_Molex:Molex_PicoBlade_53048-0410_1x04_P1.25mm_Horizontal -> Connector_Molex:Molex_Panelmate_53780-0470_1x04-1MP_P1.25mm_Horizontal
Other:
- sheet STM1_CAN ports: added USB_D+, USB_D-; removed USB_DM, USB_DP
- sheet STM2_CAN ports: added USB_D+, USB_D-; removed USB_DM, USB_DP
Changed lines of the file:
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@@
       (effects (font (size 1.27 1.27)) hide)
     )
-    (property "Footprint" "Connector_Molex:Molex_PicoBlade_53048-0410_1x04_P1.25mm_Horizontal" (id 2) (at 84.582 85.09 0)
+    (property "Footprint" "Connector_Molex:Molex_Panelmate_53780-0470_1x04-1MP_P1.25mm_Horizontal" (id 2) (at 84.582 85.09 0)
       (effects (font (size 1.27 1.27)) hide)
     )
@@
       (effects (font (size 1.27 1.27)) (justify left top) hide)
     )
-    (pin "USB_DP" bidirectional (at 147.066 112.268 180)
-      (effects (font (size 1.27 1.27)) (justify left))
-    )
-    (pin "USB_DM" bidirectional (at 147.066 109.728 180)
-      (effects (font (size 1.27 1.27)) (justify left))
-    )
     (pin "CAN_L" bidirectional (at 164.592 112.268 0)
       (effects (font (size 1.27 1.27)) (justify right))
@@
     (pin "CAN_H" bidirectional (at 164.592 109.728 0)
       (effects (font (size 1.27 1.27)) (justify right))
+    )
+    (pin "USB_D-" bidirectional (at 147.066 109.728 180)
+      (effects (font (size 1.27 1.27)) (justify left))
+    )
+    (pin "USB_D+" bidirectional (at 147.066 112.268 180)
+      (effects (font (size 1.27 1.27)) (justify left))
     )
   )
@@
       (effects (font (size 1.27 1.27)) (justify left top) hide)
     )
-    (pin "USB_DP" bidirectional (at 147.066 124.206 180)
-      (effects (font (size 1.27 1.27)) (justify left))
-    )
-    (pin "USB_DM" bidirectional (at 147.066 121.666 180)
-      (effects (font (size 1.27 1.27)) (justify left))
-    )
     (pin "CAN_L" bidirectional (at 164.338 124.206 0)
       (effects (font (size 1.27 1.27)) (justify right))
@@
     (pin "CAN_H" bidirectional (at 164.338 121.666 0)
       (effects (font (size 1.27 1.27)) (justify right))
+    )
+    (pin "USB_D-" bidirectional (at 147.066 121.666 180)
+      (effects (font (size 1.27 1.27)) (justify left))
+    )
+    (pin "USB_D+" bidirectional (at 147.066 124.206 180)
+      (effects (font (size 1.27 1.27)) (justify left))
     )
   )
@@
       (reference "#PWR034") (unit 1) (value "GND") (footprint "")
     )
-    (path "/863ee6bd-9a8e-49fb-84d6-8d00fe76baf1/655fcadd-68be-4ec1-b070-858ca61166ea"
-      (reference "#PWR035") (unit 1) (value "VCC") (footprint "")
-    )
-    (path "/863ee6bd-9a8e-49fb-84d6-8d00fe76baf1/a30fb8c9-05d6-46dc-bc65-ac4f5e35ccd1"
-      (reference "#PWR036") (unit 1) (value "GND") (footprint "")
-    )
-    (path "/9b90d3c5-a48b-42a5-8d7c-de34d4b66dbc/5784f0ea-0d0f-4a00-beeb-c20d277e2803"
-      (reference "#PWR037") (unit 1) (value "VCC") (footprint "")
-    )
-    (path "/9b90d3c5-a48b-42a5-8d7c-de34d4b66dbc/1528ec23-0172-4ce4-b199-19e9aa5f9b8d"
-      (reference "#PWR038") (unit 1) (value "GND") (footprint "")
-    )
     (path "/863ee6bd-9a8e-49fb-84d6-8d00fe76baf1/e4e7f92b-762c-4d66-a27a-28f122ae3c86"
       (reference "#PWR0101") (unit 1) (value "VCC") (footprint "")
@@
     )
     (path "/3d353840-3aaf-44c3-860e-5387613b4726"
-      (reference "J1") (unit 1) (value "Conn_01x04") (footprint "Connector_Molex:Molex_PicoBlade_53048-0410_1x04_P1.25mm_Horizontal")
+      (reference "J1") (unit 1) (value "Conn_01x04") (footprint "Connector_Molex:Molex_Panelmate_53780-0470_1x04-1MP_P1.25mm_Horizontal")
     )
     (path "/e547fe25-99ba-4e40-b44f-26baa2850f1a"
@@
       (reference "J5") (unit 1) (value "Conn_01x02") (footprint "Connector_JST:JST_GH_SM02B-GHS-TB_1x02-1MP_P1.25mm_Horizontal")
     )
-    (path "/863ee6bd-9a8e-49fb-84d6-8d00fe76baf1/d052fbd0-3edb-438a-9023-a492dd381006"
-      (reference "J6") (unit 1) (value "Conn_01x04") (footprint "Connector_JST:JST_GH_BM04B-GHS-TBT_1x04-1MP_P1.25mm_Vertical")
-    )
-    (path "/9b90d3c5-a48b-42a5-8d7c-de34d4b66dbc/a4956195-9595-410b-8691-21adeee0fc23"
-      (reference "J7") (unit 1) (value "Conn_01x04") (footprint "Connector_JST:JST_GH_BM04B-GHS-TBT_1x04-1MP_P1.25mm_Vertical")
-    )
-    (path "/71b07c00-0314-4dfd-92cb-aca2c9812e1b/0322e890-da8e-42af-9b88-ae693ad0c229"
+    (path "/71b07c00-0314-4dfd-92cb-aca2c9812e1b/e5588e62-caec-4581-8753-afa8055836e7"
       (reference "Q1") (unit 1) (value "S8050") (footprint "Package_TO_SOT_SMD:SOT-23")
     )

Commit message: update MX1.25 seat
Parts:
- J1: footprint Connector_Molex:Molex_Panelmate_53780-0470_1x04-1MP_P1.25mm_Horizontal -> Connector_Molex:Molex_CLIK-Mate_502386-0470_1x04-1MP_P1.25mm_Horizontal
Changed lines of the file:
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@@
       (effects (font (size 1.27 1.27)) hide)
     )
-    (property "Footprint" "Connector_Molex:Molex_Panelmate_53780-0470_1x04-1MP_P1.25mm_Horizontal" (id 2) (at 84.582 85.09 0)
+    (property "Footprint" "Connector_Molex:Molex_CLIK-Mate_502386-0470_1x04-1MP_P1.25mm_Horizontal" (id 2) (at 84.582 85.09 0)
       (effects (font (size 1.27 1.27)) hide)
     )
@@
     )
     (path "/3d353840-3aaf-44c3-860e-5387613b4726"
-      (reference "J1") (unit 1) (value "Conn_01x04") (footprint "Connector_Molex:Molex_Panelmate_53780-0470_1x04-1MP_P1.25mm_Horizontal")
+      (reference "J1") (unit 1) (value "Conn_01x04") (footprint "Connector_Molex:Molex_CLIK-Mate_502386-0470_1x04-1MP_P1.25mm_Horizontal")
     )
     (path "/e547fe25-99ba-4e40-b44f-26baa2850f1a"
